File: FlatMonitorv3/FlatMonitorv3.kicad_pcb (KiCad board)
At the start: 2 copper layers, 4 parts, among them J1 RJ45, U1 STM32F107VCTx, U2 BMP280, U3 BMP280

Commit message: PCB in progress
Parts:
- removed U3: BMP280, Display:OLED-128O064D
- added J2: USB_B_Micro, Connector_USB:USB_Micro-B_Amphenol_10104110_Horizontal, F.Cu at (125.2, 62.7)
- added U4: BMP280, Package_LGA:Bosch_LGA-8_2x2.5mm_P0.65mm_ClockwisePinNumbering, F.Cu at (143.2, 60.8)
Connections:
- U2 pad 2: unconnected-(U2-CSB-Pad2) -> Net-(U2-CSB)
- U2 pad 3: unconnected-(U2-SDI-Pad3) -> Net-(U2-SDI)
- U2 pad 4: unconnected-(U2-SCK-Pad4) -> Net-(U2-SCK)
- U2 pad 5: unconnected-(U2-SDO-Pad5) -> Net-(U2-SDO)
