File: FlatMonitorv3/FlatMonitorv3.kicad_sch (KiCad schematic)
At the start: 5 parts, among them J1 RJ45, J2 USB_B_Micro, U1 STM32F107VCTx, U2 BMP280, U4 BMP280

Commit message: firmware init
Connections:
- net at J2.2 (D-): now also U1.78 (PC10)
- net at J2.3 (D+): now also U1.79 (PC11)
Other:
- moved on the sheet: J2
Changed lines of the file:
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@@
+	(wire
+		(pts
+			(xy 152.4 143.51) (xy 177.8 143.51)
+		)
+		(stroke
+			(width 0)
+			(type default)
+		)
+	)
 	(wire
 		(pts
 			(xy 35.56 154.94) (xy 35.56 147.32)
+		)
+		(stroke
+			(width 0)
+			(type default)
+		)
+	)
+	(wire
+		(pts
+			(xy 152.4 140.97) (xy 177.8 140.97)
 		)
 		(stroke
@@
 	(symbol
 		(lib_id "Connector:USB_B_Micro")
-		(at 185.42 124.46 180)
+		(at 185.42 143.51 180)
 		(unit 1)
 		(exclude_from_sim no)
@@
 		(fields_autoplaced yes)
 		(property "Reference" "J2"
-			(at 191.77 123.1899 0)
+			(at 191.77 142.2399 0)
 			(effects
 				(font
@@
 		)
 		(property "Value" "USB_B_Micro"
-			(at 191.77 125.7299 0)
+			(at 191.77 144.7799 0)
 			(effects
 				(font
@@
 		)
 		(property "Footprint" "Connector_USB:USB_Micro-B_Amphenol_10104110_Horizontal"
-			(at 181.61 123.19 0)
+			(at 181.61 142.24 0)
 			(effects
 				(font
@@
 		)
 		(property "Datasheet" "~"
-			(at 181.61 123.19 0)
+			(at 181.61 142.24 0)
 			(effects
 				(font
@@
 		)
 		(property "Description" "USB Micro Type B connector"
-			(at 185.42 124.46 0)
+			(at 185.42 143.51 0)
 			(effects
 				(font
